Commit message: base above ground, links on ground

File: urdf/triorb.urdf (robot description, URDF)
Before this commit: robot triorb, 6 links, 5 joints
Joints:
- joint base_mount_joint: origin xyz=0 0 0 rpy=0 0 0 -> xyz=0 0 0.30 rpy=0 0 0

Commit message: rename world to odom

File: urdf/triorb.urdf (robot description, URDF)
Before this commit: robot triorb, 6 links, 5 joints
Links:
- removed link world
- added link odom
Joints:
- joint base_x: parent world -> odom
