Commit message: rotation applied on mout link

File: urdf/triorb.urdf (robot description, URDF)
Before this commit: robot triorb, 6 links, 5 joints
Joints:
- joint base_to_mount: origin xyz=0 0 0.30 rpy=0 0 0 -> xyz=0 0 0.30 rpy=0 0 -1.57079632679

Commit message: mount link rotated

File: urdf/triorb.urdf (robot description, URDF)
Before this commit: robot triorb, 6 links, 5 joints
Joints:
- joint base_to_mount: origin xyz=0 0 0.30 rpy=0 0 -1.57079632679 -> xyz=0 0 0.30 rpy=0 0 -3.14159265358

Commit message: again rotated

File: urdf/triorb.urdf (robot description, URDF)
Before this commit: robot triorb, 6 links, 5 joints
Joints:
- joint base_to_mount: origin xyz=0 0 0.30 rpy=0 0 -3.14159265358 -> xyz=0 0 0.30 rpy=0 0 0
